File: hardware/front board/Sensor.kicad_sch (KiCad schematic)
At the start: 3 parts, among them IC1 VCNT2020

Commit message: front board layout & routing mostly done
Other:
- moved on the sheet: R1
Changed lines of the file:
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@@
-    (stroke (width 0) (type default))
-  )
-  (wire (pts (xy 149.86 105.41) (xy 147.32 105.41))
     (stroke (width 0) (type default))
   )
@@
     (stroke (width 0) (type default))
   )
-  (wire (pts (xy 149.86 105.41) (xy 149.86 107.95))
-    (stroke (width 0) (type default))
-  )
-  (wire (pts (xy 160.02 100.33) (xy 157.48 100.33))
+  (wire (pts (xy 149.86 100.33) (xy 149.86 97.79))
+    (stroke (width 0) (type default))
+  )
+  (wire (pts (xy 160.02 105.41) (xy 157.48 105.41))
     (stroke (width 0) (type default))
   )
@@
     (stroke (width 0) (type default))
   )
-  (wire (pts (xy 160.02 97.79) (xy 160.02 100.33))
-    (stroke (width 0) (type default))
-  )
-  (wire (pts (xy 152.4 100.33) (xy 147.32 100.33))
+  (wire (pts (xy 160.02 107.95) (xy 160.02 105.41))
+    (stroke (width 0) (type default))
+  )
+  (wire (pts (xy 152.4 105.41) (xy 147.32 105.41))
+    (stroke (width 0) (type default))
+  )
+  (wire (pts (xy 147.32 100.33) (xy 149.86 100.33))
     (stroke (width 0) (type default))
   )
@@
     (stroke (width 0) (type default))
   )
-  (label "A" (at 149.86 100.33 0) (fields_autoplaced)
+  (label "A" (at 149.86 105.41 0) (fields_autoplaced)
     (effects (font (size 0.635 0.635)) (justify left bottom))
   )
@@
     )
   )
-  (symbol (lib_id "power:+3.3V") (at 160.02 97.79 0) (unit 1)
+  (symbol (lib_id "power:+3.3V") (at 160.02 107.95 180) (unit 1)
     (in_bom yes) (on_board yes) (dnp no)
-    (property "Reference" "#PWR06" (at 160.02 101.6 0)
-      (effects (font (size 1.27 1.27)) hide)
-    )
-    (property "Value" "+3.3V" (at 160.02 93.98 0)
-      (effects (font (size 1.27 1.27)))
-    )
-    (property "Footprint" "" (at 160.02 97.79 0)
-      (effects (font (size 1.27 1.27)) hide)
-    )
-    (property "Datasheet" "" (at 160.02 97.79 0)
+    (property "Reference" "#PWR06" (at 160.02 104.14 0)
+      (effects (font (size 1.27 1.27)) hide)
+    )
+    (property "Value" "+3.3V" (at 160.02 111.76 0)
+      (effects (font (size 1.27 1.27)))
+    )
+    (property "Footprint" "" (at 160.02 107.95 0)
+      (effects (font (size 1.27 1.27)) hide)
+    )
+    (property "Datasheet" "" (at 160.02 107.95 0)
       (effects (font (size 1.27 1.27)) hide)
     )
@@
     )
   )
-  (symbol (lib_id "Device:R_Small") (at 154.94 100.33 90) (mirror x) (unit 1)
+  (symbol (lib_id "Device:R_Small") (at 154.94 105.41 90) (mirror x) (unit 1)
     (in_bom yes) (on_board yes) (dnp no) (fields_autoplaced)
-    (property "Reference" "R1" (at 154.94 95.25 90)
-      (effects (font (size 1.27 1.27)))
-    )
-    (property "Value" "100" (at 154.94 97.79 90)
-      (effects (font (size 1.27 1.27)))
-    )
-    (property "Footprint" "Resistor_SMD:R_0603_1608Metric" (at 154.94 100.33 0)
-      (effects (font (size 1.27 1.27)) hide)
-    )
-    (property "Datasheet" "~" (at 154.94 100.33 0)
+    (property "Reference" "R1" (at 154.94 100.33 90)
+      (effects (font (size 1.27 1.27)))
+    )
+    (property "Value" "100" (at 154.94 102.87 90)
+      (effects (font (size 1.27 1.27)))
+    )
+    (property "Footprint" "Resistor_SMD:R_0603_1608Metric" (at 154.94 105.41 0)
+      (effects (font (size 1.27 1.27)) hide)
+    )
+    (property "Datasheet" "~" (at 154.94 105.41 0)
       (effects (font (size 1.27 1.27)) hide)
     )
@@
     )
   )
-  (symbol (lib_id "power:GND") (at 149.86 107.95 0) (mirror y) (unit 1)
+  (symbol (lib_id "power:GND") (at 149.86 97.79 0) (mirror x) (unit 1)
     (in_bom yes) (on_board yes) (dnp no)
-    (property "Reference" "#PWR041" (at 149.86 114.3 0)
-      (effects (font (size 1.27 1.27)) hide)
-    )
-    (property "Value" "GND" (at 149.86 111.76 0)
-      (effects (font (size 1.27 1.27)))
-    )
-    (property "Footprint" "" (at 149.86 107.95 0)
-      (effects (font (size 1.27 1.27)) hide)
-    )
-    (property "Datasheet" "" (at 149.86 107.95 0)
-      (effects (font (size 1.27 1.27)) hide)
-    )
+    (property "Reference" "#PWR041" (at 149.86 91.44 0)
+      (effects (font (size 1.27 1.27)) hide)
+    )
+    (property "Value" "GND" (at 149.86 93.98 0)
+      (effects (font (size 1.27 1.27)))
+    )
+    (property "Footprint" "" (at 149.86 97.79 0)
+      (effects (font (size 1.27 1.27)) hide)
+    )
+    (property "Datasheet" "" (at 149.86 97.79 0)
+      (effects (font (size 1.27 1.27)) hide)
+    )
