File: hardware/front board/SmSemProject-FrontBoard.kicad_pcb (KiCad board)
At the start: 2 copper layers, 58 parts, among them IC1 VCNT2020, IC10 VCNT2020, IC11 VCNT2020, IC12 VCNT2020, IC13 VCNT2020, IC14 VCNT2020, IC15 VCNT2020, IC16 VCNT2020, IC17 VCNT2020, IC2 MAX11643EEG+, IC3 VCNT2020, IC4 VCNT2020, IC5 VCNT2020, IC6 VCNT2020, IC7 VCNT2020, IC8 VCNT2020, IC9 VCNT2020, J1 Conn_01x10

Commit message: front board layout & routing mostly done
Parts:
- removed J1: Conn_01x10, Connector_FFC-FPC:Molex_200528-0100_1x10-1MP_P1.00mm_Horizontal
- added J2: Conn_01x10_MountingPin, Connector_FFC-FPC:Molex_200528-0100_1x10-1MP_P1.00mm_Horizontal, F.Cu at (141.5, 74.6)
- C1, C2, IC1, IC10, IC11, IC12, IC13, IC14, IC15, IC16, IC17, IC3, IC4, IC5, IC6, IC7, IC8, IC9, R1, R10, R11, R12, R13, R14, R15, R16, R17, R18, R19, R2, R20, R21, R22, R23, R24, R25, R26, R27, R28, R29, R3, R30, R31, R32, R33, R34, R4, R5, R6, R7, R8, R9: moved to B.Cu
- moved R32 109.6 mm to (76.5, 75.4), turned to 180 degrees
- moved R22 109.2 mm to (126.5, 65.1), turned to 180 degrees
- moved R14 108.7 mm to (166.5, 66.1), turned to 180 degrees
- moved IC17 107.6 mm to (76.5, 77.9), turned to 90 degrees
- moved R18 106.8 mm to (106.5, 67.6), turned to 180 degrees
- moved R30 105.2 mm to (86.5, 72.2), turned to 180 degrees
- moved IC12 104.3 mm to (126.5, 67.6), turned to 90 degrees
- moved IC10 104.2 mm to (106.5, 70.1), turned to 90 degrees
- moved IC16 103.9 mm to (86.5, 74.7), turned to 90 degrees
- moved R10 103.6 mm to (146.5, 64.5), turned to 180 degrees
- moved IC8 102.9 mm to (166.5, 68.6), turned to 90 degrees
- moved R31 102.9 mm to (76.5, 80.4), turned to 180 degrees
- moved H4 101.8 mm to (161.5, 65.5)
- moved R28 101.8 mm to (96.5, 69.6), turned to 180 degrees
- moved R13 101.8 mm to (166.5, 71.1), turned to 180 degrees
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Connections:
- IC2 pad 23: /SPI_MOSI -> /SPI_MISO
Routing:
- net /OUT0: track 0.00 -> 84.9 mm, vias 0 -> 1
- net /OUT15: track 0.00 -> 80.4 mm, vias 0 -> 1
- net /OUT1: track 0.00 -> 73.4 mm, vias 0 -> 1
- net /OUT14: track 0.00 -> 68.2 mm, vias 0 -> 1
- net /OUT2: track 0.00 -> 62.7 mm, vias 0 -> 1
- net /OUT13: track 0.00 -> 55.1 mm, vias 0 -> 1
- net /OUT3: track 0.00 -> 52.4 mm, vias 0 -> 1
- net /OUT12: track 0.00 -> 45.3 mm, vias 0 -> 1
- net /OUT4: track 0.00 -> 43.2 mm, vias 0 -> 1
- net /OUT11: track 0.00 -> 37.1 mm, vias 0 -> 1
- net /OUT5: track 0.00 -> 33.6 mm, vias 0 -> 1
- net /OUT10: track 0.00 -> 26.8 mm, vias 0 -> 1
- net /OUT6: track 0.00 -> 24.2 mm, vias 0 -> 1
- net /OUT9: track 0.00 -> 16.5 mm, vias 0 -> 1
- net /SPI_EX_INT1: track 0.00 -> 16.2 mm
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- added copper zone on B.Cu, net GND
- added copper zone on F.Cu, net GND
Other:
- board outline added: 166.9 x 27.6 mm

Commit message: all layouts and routings done
Parts:
- moved C1 3.42 mm to (142.3, 70.2), turned to 90 degrees
- moved C2 3.42 mm to (140.7, 70.2), turned to 90 degrees
Routing:
- net +3.3V: track 8.29 -> 279.3 mm, vias 3 -> 34
- net /OUT1: track 73.4 -> 81.6 mm, vias 1 -> 3
- net /OUT2: track 62.7 -> 70.2 mm, vias 1 -> 3
- net GND: track 0.00 -> 2.71 mm, vias 5 -> 452
- net /OUT3: track 52.4 -> 53.7 mm
- net /OUT6: track 24.2 -> 25.5 mm
- net /OUT13: track 55.1 -> 56.2 mm
- net /OUT12: track 45.3 -> 44.4 mm
- net /OUT10: track 26.8 -> 27.7 mm
- net /OUT11: track 37.1 -> 36.2 mm
- net /OUT9: track 16.5 -> 17.3 mm
- net /OUT5: track 33.6 -> 34.5 mm
- net /OUT4: track 43.2 -> 43.9 mm
- net /OUT0: track 84.9 -> 85.5 mm
