File: hardware/front board/SmSemProject-FrontBoard.kicad_sch (KiCad schematic)
At the start: 10 parts, among them IC2 MAX11643EEG+, J7 Conn_01x10

Commit message: front board layout & routing mostly done
Parts:
- removed J7: Conn_01x10, Connector_FFC-FPC:Molex_200528-0100_1x10-1MP_P1.00mm_Horizontal, symbol Connector_Generic:Conn_01x10
- added J2: Conn_01x10_MountingPin, Connector_FFC-FPC:Molex_200528-0100_1x10-1MP_P1.00mm_Horizontal, symbol Connector_Generic_MountingPin:Conn_01x10_MountingPin
Connections:
- net +3.3V: now also J2.1 (Pin_1)
- net GND: now also J2.10 (Pin_10), J2.7 (Pin_7), J2.MP (MountPin)
- net SPI_CLK: now also J2.6 (Pin_6)
- net SPI_EX_INT1: now also J2.3 (Pin_3)
- net SPI_MISO: now also IC2.23 (DOUT), J2.9 (Pin_9)
- net SPI_MOSI: now also J2.8 (Pin_8); no longer IC2.23 (DOUT)
- net ~{SPI_EX1_CS}: now also J2.5 (Pin_5)
Changed lines of the file:
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@@
+    (stroke (width 0) (type default))
+  )
+  (wire (pts (xy 125.73 78.74) (xy 128.27 78.74))
     (stroke (width 0) (type default))
   )
@@
     (stroke (width 0) (type default))
   )
+  (wire (pts (xy 125.73 76.2) (xy 128.27 76.2))
+    (stroke (width 0) (type default))
+  )
   (wire (pts (xy 105.41 76.2) (xy 105.41 78.74))
     (stroke (width 0) (type default))
@@
   )
   (wire (pts (xy 186.69 101.6) (xy 168.91 101.6))
+    (stroke (width 0) (type default))
+  )
+  (wire (pts (xy 46.99 73.66) (xy 46.99 76.2))
     (stroke (width 0) (type default))
   )
@@
     (effects (font (size 1.27 1.27)) (justify left bottom))
   )
-  (label "SPI_MOSI" (at 128.27 78.74 180) (fields_autoplaced)
+  (label "SPI_MOSI" (at 125.73 78.74 180) (fields_autoplaced)
     (effects (font (size 1.27 1.27)) (justify right bottom))
   )
@@
     (effects (font (size 1.27 1.27)) (justify left bottom))
   )
-  (label "SPI_MOSI" (at 128.27 76.2 180) (fields_autoplaced)
-    (effects (font (size 1.27 1.27)) (justify right bottom))
-  )
   (label "OUT10" (at 171.45 99.06 0) (fields_autoplaced)
     (effects (font (size 1.27 1.27)) (justify left bottom))
@@
   )
   (label "OUT15" (at 125.73 93.98 180) (fields_autoplaced)
+    (effects (font (size 1.27 1.27)) (justify right bottom))
+  )
+  (label "SPI_MISO" (at 125.73 76.2 180) (fields_autoplaced)
     (effects (font (size 1.27 1.27)) (justify right bottom))
   )
@@
     )
   )
-  (symbol (lib_id "Device:C_Small") (at 105.41 81.28 0) (mirror y) (unit 1)
-    (in_bom yes) (on_board yes) (dnp no)
-    (property "Reference" "C13" (at 100.33 82.55 0)
-      (effects (font (size 1.27 1.27)))
-    )
-    (property "Value" "100nF" (at 100.33 80.01 0)
-      (effects (font (size 1.27 1.27)))
-    )
-    (property "Footprint" "Capacitor_SMD:C_0603_1608Metric" (at 105.41 81.28 0)
-      (effects (font (size 1.27 1.27)) hide)
-    )
-    (property "Datasheet" "~" (at 105.41 81.28 0)
-      (effects (font (size 1.27 1.27)) hide)
-    )
-    (property "Manufacturer_Name" "--" (at 105.41 81.28 0)
-      (effects (font (size 1.27 1.27)) hide)
-    )
-    (property "Manufacturer_Part_Number" "--" (at 105.41 81.28 0)
-      (effects (font (size 1.27 1.27)) hide)
-    )
-    (pin "1")
-    (pin "2")
-    (instances
-      (project "SmSemProject"
-        (path "/2d1fee9c-ff28-4ed3-bed9-80ad18eb590f/f72e7ef6-ff36-4e66-b7fe-270099ead489"
-          (reference "C13") (unit 1)
-        )
-        (path "/2d1fee9c-ff28-4ed3-bed9-80ad18eb590f"
-          (reference "C27") (unit 1)
-        )
-      )
-      (project "SmSemProject-FrontBoard"
-        (path "/62cf8cd9-1bcb-4159-b3f1-7d9a95a75f08"
-          (reference "C1") (unit 1)
-        )
-      )
-      (project "PUTM_EV_BMS_HV_Master_2021"
-        (path "/b456cffc-d9d7-4c91-91f2-36ec9a65dd1b/e61cc821-5479-4c04-b5ab-4a32f17b4f03/d2e30d51-b8f8-4bbd-bb5a-76e0eb119260"
-          (reference "C7") (unit 1)
-        )
-        (path "/b456cffc-d9d7-4c91-91f2-36ec9a65dd1b/e61cc821-5479-4c04-b5ab-4a32f17b4f03/6b03d8c8-5f6c-4244-9202-23821031eb5e"
-          (reference "C22") (unit 1)
-        )
-        (path "/b456cffc-d9d7-4c91-91f2-36ec9a65dd1b/e61cc821-5479-4c04-b5ab-4a32f17b4f03"
-          (reference "C26") (unit 1)
-        )
-      )
-    )
-  )
-  (symbol (lib_id "power:+3.3V") (at 91.44 86.36 90) (unit 1)
-    (in_bom yes) (on_board yes) (dnp no)
-    (property "Reference" "#PWR06" (at 95.25 86.36 0)
-      (effects (font (size 1.27 1.27)) hide)
-    )
-    (property "Value" "+3.3V" (at 85.09 86.36 90)
-      (effects (font (size 1.27 1.27)))
-    )
-    (property "Footprint" "" (at 91.44 86.36 0)
-      (effects (font (size 1.27 1.27)) hide)
-    )
-    (property "Datasheet" "" (at 91.44 86.36 0)
-      (effects (font (size 1.27 1.27)) hide)
-    )
-    (pin "1")
-    (instances
-      (project "SmSemProject"
-        (path "/2d1fee9c-ff28-4ed3-bed9-80ad18eb590f/f72e7ef6-ff36-4e66-b7fe-270099ead489"
-          (reference "#PWR06") (unit 1)
-        )
-        (path "/2d1fee9c-ff28-4ed3-bed9-80ad18eb590f"
-          (reference "#PWR040") (unit 1)
-        )
-      )
-      (project "SmSemProject-FrontBoard"
-        (path "/62cf8cd9-1bcb-4159-b3f1-7d9a95a75f08"
-          (reference "#PWR04") (unit 1)
-        )
-      )
-    )
-  )
-  (symbol (lib_id "Connector_Generic:Conn_01x10") (at 46.99 55.88 0) (mirror y) (unit 1)
-    (in_bom yes) (on_board yes) (dnp no)
-    (property "Reference" "J7" (at 44.45 56.515 0)
-      (effects (font (size 1.27 1.27)) (justify left))
-    )
-    (property "Value" "Conn_01x10" (at 44.45 59.055 0)
-      (effects (font (size 1.27 1.27)) (justify left))
+  (symbol (lib_id "Connector_Generic_MountingPin:Conn_01x10_MountingPin") (at 46.99 55.88 0) (mirror y) (unit 1)
+    (in_bom yes) (on_board yes) (dnp no) (fields_autoplaced)
+    (property "Reference" "J2" (at 46.99 39.37 0)
+      (effects (font (size 1.27 1.27)))
+    )
+    (property "Value" "Conn_01x10_MountingPin" (at 46.99 41.91 0)
+      (effects (font (size 1.27 1.27)))
     )
     (property "Footprint" "Connector_FFC-FPC:Molex_200528-0100_1x10-1MP_P1.00mm_Horizontal" (at 46.99 55.88 0)
@@
     (pin "8")
     (pin "9")
-    (instances
-      (project "SmSemProject"
-        (path "/2d1fee9c-ff28-4ed3-bed9-80ad18eb590f"
-          (reference "J7") (unit 1)
-        )
-      )
-      (project "SmSemProject-FrontBoard"
-        (path "/62cf8cd9-1bcb-4159-b3f1-7d9a95a75f08"
-          (reference "J1") (unit 1)
+    (pin "MP")
+    (instances
+      (project "SmSemProject-FrontBoard"
+        (path "/62cf8cd9-1bcb-4159-b3f1-7d9a95a75f08"
+          (reference "J2") (unit 1)
+        )
+      )
+    )
+  )
+  (symbol (lib_id "Device:C_Small") (at 105.41 81.28 0) (mirror y) (unit 1)
+    (in_bom yes) (on_board yes) (dnp no)
+    (property "Reference" "C13" (at 100.33 82.55 0)
+      (effects (font (size 1.27 1.27)))
+    )
+    (property "Value" "100nF" (at 100.33 80.01 0)
+      (effects (font (size 1.27 1.27)))
+    )
+    (property "Footprint" "Capacitor_SMD:C_0603_1608Metric" (at 105.41 81.28 0)
+      (effects (font (size 1.27 1.27)) hide)
+    )
+    (property "Datasheet" "~" (at 105.41 81.28 0)
+      (effects (font (size 1.27 1.27)) hide)
+    )
+    (property "Manufacturer_Name" "--" (at 105.41 81.28 0)
+      (effects (font (size 1.27 1.27)) hide)
+    )
+    (property "Manufacturer_Part_Number" "--" (at 105.41 81.28 0)
+      (effects (font (size 1.27 1.27)) hide)
+    )
+    (pin "1")
+    (pin "2")
+    (instances
+      (project "SmSemProject"
+        (path "/2d1fee9c-ff28-4ed3-bed9-80ad18eb590f/f72e7ef6-ff36-4e66-b7fe-270099ead489"
+          (reference "C13") (unit 1)
+        )
+        (path "/2d1fee9c-ff28-4ed3-bed9-80ad18eb590f"
+          (reference "C27") (unit 1)
+        )
+      )
+      (project "SmSemProject-FrontBoard"
+        (path "/62cf8cd9-1bcb-4159-b3f1-7d9a95a75f08"
+          (reference "C1") (unit 1)
+        )
+      )
+      (project "PUTM_EV_BMS_HV_Master_2021"
+        (path "/b456cffc-d9d7-4c91-91f2-36ec9a65dd1b/e61cc821-5479-4c04-b5ab-4a32f17b4f03/d2e30d51-b8f8-4bbd-bb5a-76e0eb119260"
+          (reference "C7") (unit 1)
+        )
+        (path "/b456cffc-d9d7-4c91-91f2-36ec9a65dd1b/e61cc821-5479-4c04-b5ab-4a32f17b4f03/6b03d8c8-5f6c-4244-9202-23821031eb5e"
+          (reference "C22") (unit 1)
+        )
+        (path "/b456cffc-d9d7-4c91-91f2-36ec9a65dd1b/e61cc821-5479-4c04-b5ab-4a32f17b4f03"
+          (reference "C26") (unit 1)
+        )
+      )
+    )
+  )
+  (symbol (lib_id "power:+3.3V") (at 91.44 86.36 90) (unit 1)
+    (in_bom yes) (on_board yes) (dnp no)
+    (property "Reference" "#PWR06" (at 95.25 86.36 0)
+      (effects (font (size 1.27 1.27)) hide)
+    )
+    (property "Value" "+3.3V" (at 85.09 86.36 90)
+      (effects (font (size 1.27 1.27)))
+    )
+    (property "Footprint" "" (at 91.44 86.36 0)
+      (effects (font (size 1.27 1.27)) hide)
+    )
+    (property "Datasheet" "" (at 91.44 86.36 0)
+      (effects (font (size 1.27 1.27)) hide)
+    )
+    (pin "1")
+    (instances
+      (project "SmSemProject"
+        (path "/2d1fee9c-ff28-4ed3-bed9-80ad18eb590f/f72e7ef6-ff36-4e66-b7fe-270099ead489"
+          (reference "#PWR06") (unit 1)
+        )
+        (path "/2d1fee9c-ff28-4ed3-bed9-80ad18eb590f"
+          (reference "#PWR040") (unit 1)
+        )
+      )
+      (project "SmSemProject-FrontBoard"
+        (path "/62cf8cd9-1bcb-4159-b3f1-7d9a95a75f08"
+          (reference "#PWR04") (unit 1)
         )
       )
@@
         )
       )
+    )
+  )
+  (symbol (lib_id "power:GND") (at 46.99 76.2 0) (unit 1)
+    (in_bom yes) (on_board yes) (dnp no)
+    (property "Reference" "#PWR041" (at 46.99 82.55 0)
+      (effects (font (size 1.27 1.27)) hide)
+    )
+    (property "Value" "GND" (at 46.99 80.01 0)
+      (effects (font (size 1.27 1.27)))
+    )
+    (property "Footprint" "" (at 46.99 76.2 0)
+      (effects (font (size 1.27 1.27)) hide)
+    )
+    (property "Datasheet" "" (at 46.99 76.2 0)
+      (effects (font (size 1.27 1.27)) hide)
+    )
+    (pin "1")
+    (instances
+      (project "SmSemProject"
+        (path "/2d1fee9c-ff28-4ed3-bed9-80ad18eb590f"
+          (reference "#PWR041") (unit 1)
+        )
+      )
+      (project "SmSemProject-FrontBoard"
+        (path "/62cf8cd9-1bcb-4159-b3f1-7d9a95a75f08"
+          (reference "#PWR072") (unit 1)
+        )
+      )

Commit message: firmware - added common classes
Parts:
- C13: Dodane do zamówienia (none) -> 1
Changed lines of the file:
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@@
+      (effects (font (size 1.27 1.27)) hide)
+    )
+    (property "Dodane do zamówienia" "" (at 66.04 177.8 0)
       (effects (font (size 1.27 1.27)) hide)
     )
@@
       (effects (font (size 1.27 1.27)) hide)
     )
+    (property "Dodane do zamówienia" "" (at 120.65 184.15 0)
+      (effects (font (size 1.27 1.27)) hide)
+    )
     (pin "1")
     (instances
@@
       (effects (font (size 1.27 1.27)) hide)
     )
+    (property "Dodane do zamówienia" "" (at 76.2 177.8 0)
+      (effects (font (size 1.27 1.27)) hide)
+    )
     (pin "1")
     (pin "2")
@@
     )
     (property "Manufacturer_Part_Number" "--" (at 93.98 81.28 0)
+      (effects (font (size 1.27 1.27)) hide)
+    )
+    (property "Dodane do zamówienia" "1" (at 93.98 81.28 0)
       (effects (font (size 1.27 1.27)) hide)
     )
@@
       (effects (font (size 1.27 1.27)) hide)
     )
+    (property "Dodane do zamówienia" "" (at 120.65 172.72 0)
+      (effects (font (size 1.27 1.27)) hide)
+    )
     (pin "1")
     (instances
@@
     )
     (property "Datasheet" "~" (at 140.97 184.15 0)
+      (effects (font (size 1.27 1.27)) hide)
+    )
+    (property "Dodane do zamówienia" "" (at 140.97 184.15 0)
       (effects (font (size 1.27 1.27)) hide)
     )
@@
     )
     (property "Datasheet" "~" (at 46.99 55.88 0)
+      (effects (font (size 1.27 1.27)) hide)
+    )
+    (property "Dodane do zamówienia" "" (at 46.99 55.88 0)
       (effects (font (size 1.27 1.27)) hide)
     )
@@
       (effects (font (size 1.27 1.27)) hide)
     )
+    (property "Dodane do zamówienia" "1" (at 105.41 81.28 0)
+      (effects (font (size 1.27 1.27)) hide)
+    )
     (pin "1")
     (pin "2")
@@
       (effects (font (size 1.27 1.27)) hide)
     )
+    (property "Dodane do zamówienia" "" (at 140.97 172.72 0)
+      (effects (font (size 1.27 1.27)) hide)
+    )
     (pin "1")
     (instances
@@
       (effects (font (size 1.27 1.27)) (justify left top) hide)
     )
-    (pin "1")
+    (property "Dodane do zamówienia" "" (at 148.59 87.63 0)
+      (effects (font (size 1.27 1.27)) hide)
+    )
+    (pin "1")
