File: hardware/main board/MotorControl.kicad_sch (KiCad schematic)
At the start: 3 parts, among them IC2 DRV8212PDSGR

Commit message: all layouts and routings done
Parts:
- added C19: 100nF, Capacitor_SMD:C_0603_1608Metric, symbol Device:C_Small
- added IC6: SN74LVC1G18DBVRG4, Package_TO_SOT_SMD:SOT-23-6, symbol Samacsys_kicad_sym:SN74LVC1G18DBVRG4
Connections:
- net +3.3V: now also C19.1, IC6.5 (VCC)
- net GND: now also C19.2, IC6.2 (GND)
- net M+: now also IC2.3 (OUT2); no longer IC2.2 (OUT1)
- net M-: now also IC2.2 (OUT1); no longer IC2.3 (OUT2)
- net FORWARD_PWM renamed PWMF
- net PWMF: now also IC6.4
- net REVERSE_PWM renamed PWMR
- net PWMR: now also IC6.6
- new net DIRECTION: IC6.1
- new net PWM: IC6.3
Other:
- moved on the sheet: C14, C19, IC2

Commit message: firmware - added common classes
Parts:
- C14: Dodane do zamówienia (none) -> 10; Mouser Part Number (none) -> 187-CL10A475KO8NNNC; Mouser Price/Stock (none) -> https://www.mouser.pl/ProductDetail/Samsung-Electro-Mechani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
- C19: Dodane do zamówienia (none) -> 20; Mouser Part Number (none) -> 963-EMK107B7104MA-T; Mouser Price/Stock (none) -> https://www.mouser.pl/ProductDetail/TAIYO-YUDEN/EMK107B7104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
- IC2, IC6: Dodane do zamówienia (none) -> 1
Changed lines of the file:
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@@
       (effects (font (size 1.27 1.27)) (justify left top) hide)
+    )
+    (property "Dodane do zamówienia" "1" (at 113.03 87.63 0)
+      (effects (font (size 1.27 1.27)) hide)
     )
     (pin "1")
@@
       (effects (font (size 1.27 1.27)) (justify left top) hide)
     )
+    (property "Dodane do zamówienia" "1" (at 162.56 92.71 0)
+      (effects (font (size 1.27 1.27)) hide)
+    )
     (pin "1")
     (pin "2")
@@
       (effects (font (size 1.27 1.27)) hide)
     )
+    (property "Dodane do zamówienia" "20" (at 148.59 106.68 0)
+      (effects (font (size 1.27 1.27)) hide)
+    )
+    (property "Mouser Part Number" "963-EMK107B7104MA-T" (at 148.59 106.68 0)
+      (effects (font (size 1.27 1.27)) hide)
+    )
+    (property "Mouser Price/Stock" "https://www.mouser.pl/ProductDetail/TAIYO-YUDEN/EMK107B7104MA-T?qs=I6KAKw0tg2yoDM4kgVF98Q%3D%3D" (at 148.59 106.68 0)
+      (effects (font (size 1.27 1.27)) hide)
+    )
     (pin "1")
     (pin "2")
@@
       (effects (font (size 1.27 1.27)) hide)
     )
+    (property "Dodane do zamówienia" "20" (at 129.54 76.2 0)
+      (effects (font (size 1.27 1.27)) hide)
+    )
+    (property "Mouser Part Number" "963-EMK107B7104MA-T" (at 129.54 76.2 0)
+      (effects (font (size 1.27 1.27)) hide)
+    )
+    (property "Mouser Price/Stock" "https://www.mouser.pl/ProductDetail/TAIYO-YUDEN/EMK107B7104MA-T?qs=I6KAKw0tg2yoDM4kgVF98Q%3D%3D" (at 129.54 76.2 0)
+      (effects (font (size 1.27 1.27)) hide)
+    )
     (pin "1")
     (pin "2")
@@
       (effects (font (size 1.27 1.27)) hide)
     )
+    (property "Dodane do zamówienia" "10" (at 96.52 76.2 0)
+      (effects (font (size 1.27 1.27)) hide)
+    )
+    (property "Mouser Part Number" "187-CL10A475KO8NNNC" (at 96.52 76.2 0)
+      (effects (font (size 1.27 1.27)) hide)
+    )
+    (property "Mouser Price/Stock" "https://www.mouser.pl/ProductDetail/Samsung-Electro-Mechanics/CL10A475KO8NNNC?qs=X6jEic%2FHinAbIjmLnFfqqQ%3D%3D" (at 96.52 76.2 0)
+      (effects (font (size 1.27 1.27)) hide)
+    )
