File: hardware/main board/SmSemProject.kicad_pcb (KiCad board)
At the start: 8 copper layers, 50 x 50 mm, 70 parts, among them IC1 STM32WB55RGV6, IC2 DRV8212PDSGR, IC3 DRV8212PDSGR, IC4 W25N01GVZEIG, IC5 LSM6DSLTR, J1 JST-SH 01x06, J2 JST-SH 01x06, J3 JST-SH 01x03, J4 Front board out, J5 TAG CONNECT, J6 USB4145-03-0070-C, U1 LM1117MP-3.3, U2 USBLC6-2SC6, Y1 X322516MLB4SI

Commit message: front board schematic done
Parts:
- removed J4: Front board out, Connector_FFC-FPC:Molex_200528-0080_1x08-1MP_P1.00mm_Horizontal
- added J7: Conn_01x10, Connector_FFC-FPC:Molex_200528-0100_1x10-1MP_P1.00mm_Horizontal, F.Cu at (90.7, 74.2)
- moved IC1 86.2 mm to (143.5, 48.0)
- moved IC2 11.0 mm to (80.5, 83.0)

Commit message: front board layout & routing mostly done
Parts:
- moved J7 57.2 mm to (147.0, 84.1)
Connections:
- IC2 pad 2: /Motor Control Left/M+ -> /M_LEFT+
- IC2 pad 3: /Motor Control Left/M- -> /M_LEFT-
- IC3 pad 2: /Motor Control Right/M+ -> /M_LEFT+
- IC3 pad 3: /Motor Control Right/M- -> /M_LEFT-
- IC5 pad 1: /uC/SPI_MISO -> /SPI_MISO
- IC5 pad 13: /uC/SPI_CLK -> /SPI_CLK
- IC5 pad 14: /uC/SPI_MOSI -> /SPI_MOSI
- J1 pad 1: /Motor Control Right/M+ -> /M_LEFT+
- J1 pad 2: /Motor Control Right/M- -> /M_LEFT-
- J2 pad 1: /Motor Control Left/M+ -> /M_LEFT+
- J2 pad 2: /Motor Control Left/M- -> /M_LEFT-
- J2 pad 4: /M_RIGHT_A -> /M_LEFT_A
- J2 pad 5: /M_RIGHT_B -> /M_LEFT_B
- J7 pad 1: +3.3V -> GND
- J7 pad 10: GND -> +3.3V
- J7 pad 2: /uC/SPI_EX_INT1 -> /SPI_MISO
- J7 pad 3: /uC/SPI_EX_INT2 -> /SPI_MOSI
- J7 pad 4: /uC/~{SPI_EX2_CS} -> GND
- J7 pad 5: /uC/~{SPI_EX1_CS} -> /SPI_CLK
- J7 pad 6: /uC/SPI_CLK -> /~{SPI_EX1_CS}
- J7 pad 7: GND -> /~{SPI_EX2_CS}
- J7 pad 8: /uC/SPI_MOSI -> /SPI_EX_INT1
- J7 pad 9: /uC/SPI_MISO -> /SPI_EX_INT2
- J7 pad MP: (no net) -> GND
- R1 pad 2: /uC/SPI_MISO -> /SPI_MISO

Commit message: all layouts and routings done
Parts:
- removed C12: 10uF, Capacitor_SMD:C_0603_1608Metric
- removed C22, C23: 100nF, Capacitor_SMD:C_0603_1608Metric
- removed C6: 4.7uF, Capacitor_SMD:C_0603_1608Metric
- removed J5: TAG CONNECT, Connector:Tag-Connect_TC2030-IDC-FP_2x03_P1.27mm_Vertical
- removed S1: 100SP1T1B4M2QE, Samacsys:100SP1T1B4M2QE
- added C30: 100nF, Capacitor_SMD:C_0603_1608Metric, F.Cu at (163.3, 58.4)
- added C31: 100nF, Capacitor_SMD:C_0603_1608Metric, F.Cu at (130.7, 69.6)
- added D8: LED_Small, LED_SMD:LED_0603_1608Metric, F.Cu at (131.3, 61.3)
- added IC6: SN74LVC1G18DBVRG4, Package_TO_SOT_SMD:SOT-23-6, F.Cu at (160.6, 58.4)
- added IC7: SN74LVC1G18DBVRG4, Package_TO_SOT_SMD:SOT-23-6, F.Cu at (133.4, 69.6)
- added J4: FTSH-107-01-L-DV-K-A, Samacsys:FTSH-107-XX-YYY-DV-K-A, F.Cu at (166.4, 75.3)
- added R10: 10k, Resistor_SMD:R_0603_1608Metric, F.Cu at (137.2, 56.6)
- added R11: 10k, Resistor_SMD:R_0603_1608Metric, F.Cu at (138.9, 56.6)
- added R12: 10k, Resistor_SMD:R_0603_1608Metric, F.Cu at (134.5, 61.3)
- added R9: 10k, Resistor_SMD:R_0603_1608Metric, F.Cu at (140.6, 56.6)
- C26: value 100pF -> 100nF
- C27, C28, IC5: moved to B.Cu
- J3: value JST-SH 01x03 -> JST_XH_B3B; footprint Connector_JST:JST_SH_BM03B-SRSS-TB_1x03-1MP_P1.00mm_Vertical -> Connector_JST:JST_XH_B3B-XH-A_1x03_P2.50mm_Vertical
- moved J1 114.9 mm to (169.0, 64.0), turned to -90 degrees
- moved C1 112.4 mm to (159.3, 68.8), turned to 90 degrees
- moved C2 109.4 mm to (156.3, 71.5)
- moved C3 108.1 mm to (153.8, 61.0), turned to -90 degrees
- moved C16 107.2 mm to (153.7, 47.2), turned to 180 degrees
- moved R1 107.0 mm to (145.4, 56.6), turned to -90 degrees
- moved C21 106.9 mm to (148.2, 77.0)
- moved C20 106.1 mm to (148.2, 72.0), turned to 180 degrees
- moved C26 106.0 mm to (152.9, 49.9), turned to -90 degrees
- moved D1 104.7 mm to (155.8, 54.3)
- moved L3 103.4 mm to (149.0, 74.5), turned to -90 degrees
- moved C15 102.0 mm to (155.6, 61.0), turned to 90 degrees
- moved R3 101.5 mm to (131.4, 49.8)
- moved C11 101.4 mm to (149.0, 56.6), turned to -90 degrees
- moved C14 101.2 mm to (155.6, 64.4), turned to 90 degrees
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Connections:
- C29 pad 1: /VBUSFUSE -> +BATT
- D1 pad 1: /VDIODE -> +BATT
- IC1 pad 11: unconnected-(IC1A-PC2-Pad11) -> /uC/VBAT
- IC1 pad 12: unconnected-(IC1A-PC3-Pad12) -> /uC/IMU_INT1
- IC1 pad 15: unconnected-(IC1A-PA0-Pad15) -> /uC/LED1
- IC1 pad 16: unconnected-(IC1A-PA1-Pad16) -> /uC/LED2
- IC1 pad 17: unconnected-(IC1A-PA2-Pad17) -> /uC/~{QSPI_CS}
- IC1 pad 18: unconnected-(IC1A-PA3-Pad18) -> /uC/QSPI_CLK
- IC1 pad 21: unconnected-(IC1A-PA6-Pad21) -> /uC/QSPI_IO3
- IC1 pad 22: unconnected-(IC1A-PA7-Pad22) -> /uC/QSPI_IO2
- IC1 pad 23: unconnected-(IC1A-PA8-Pad23) -> /M_LEFT_PWM
- IC1 pad 24: unconnected-(IC1A-PA9-Pad24) -> /M_LEFT_DIRECTION
- IC1 pad 26: unconnected-(IC1A-PC5-Pad26) -> /uC/LED3
- IC1 pad 27: unconnected-(IC1A-PB2-Pad27) -> /uC/LED4
- IC1 pad 28: unconnected-(IC1A-PB10-Pad28) -> /uC/UART_RX
- IC1 pad 29: unconnected-(IC1A-PB11-Pad29) -> /uC/UART_TX
- IC1 pad 38: unconnected-(IC1A-PB0-Pad38) -> /Motor Control Left/~{SLEEP}
- IC1 pad 39: unconnected-(IC1A-PB1-Pad39) -> /M_RIGHT_A
- IC1 pad 40: unconnected-(IC1A-PE4-Pad40) -> /uC/IMU_INT2
- IC1 pad 50: unconnected-(IC1A-PC6-Pad50) -> /M_RIGHT_DIRECTION
- IC1 pad 51: unconnected-(IC1A-PA10-Pad51) -> /M_RIGHT_PWM
- IC1 pad 52: unconnected-(IC1A-PA11-Pad52) -> /uC/D-
- IC1 pad 53: unconnected-(IC1A-PA12-Pad53) -> /uC/D+
- IC1 pad 54: unconnected-(IC1A-PA13-Pad54) -> /uC/SWDIO
- IC1 pad 56: unconnected-(IC1A-PA14-Pad56) -> /uC/SWCLK
- IC1 pad 58: unconnected-(IC1A-PC10-Pad58) -> /~{SPI_EX1_CS}
- IC1 pad 59: unconnected-(IC1A-PC11-Pad59) -> /~{SPI_EX2_CS}
- IC1 pad 6: unconnected-(IC1A-PB8-Pad6) -> /uC/QSPI_IO1
- IC1 pad 60: unconnected-(IC1A-PC12-Pad60) -> /SPI_EX_INT1
- IC1 pad 61: unconnected-(IC1A-PD0-Pad61) -> /SPI_EX_INT2
- IC1 pad 63: unconnected-(IC1A-PB3-Pad63) -> /SPI_CLK
- IC1 pad 64: unconnected-(IC1A-PB4-Pad64) -> /SPI_MISO
- IC1 pad 65: unconnected-(IC1A-PB5-Pad65) -> /SPI_MOSI
- IC1 pad 67: unconnected-(IC1A-PB7-Pad67) -> /uC/~{SPI_IMU_CS}
- IC1 pad 7: unconnected-(IC1A-PB9-Pad7) -> /uC/QSPI_IO0
- IC1 pad 9: unconnected-(IC1A-PC0-Pad9) -> /M_LEFT_A
- IC2 pad 2: /M_LEFT+ -> /M_LEFT-
- IC2 pad 3: /M_LEFT- -> /M_LEFT+
- IC2 pad 5: /Motor Control Left/REVERSE_PWM -> /Motor Control Left/PWMR
- IC2 pad 6: /Motor Control Left/FORWARD_PWM -> /Motor Control Left/PWMF
- IC3 pad 2: /M_LEFT+ -> /M_RIGHT-
- IC3 pad 3: /M_LEFT- -> /M_RIGHT+
- IC3 pad 5: /Motor Control Right/REVERSE_PWM -> /Motor Control Right/PWMR
- IC3 pad 6: /Motor Control Right/FORWARD_PWM -> /Motor Control Right/PWMF
- J1 pad 1: /M_LEFT+ -> /M_RIGHT+
- J1 pad 2: /M_LEFT- -> /M_RIGHT-
- J1 pad 5: /M_RIGHT_B -> unconnected-(J1-Pin_5-Pad5)
- J2 pad 5: /M_LEFT_B -> unconnected-(J2-Pin_5-Pad5)
- R6 pad 1: /uC/LED1 -> /uC/LED2
- R7 pad 1: /uC/LED1 -> /uC/LED3
- R8 pad 1: /uC/LED1 -> /uC/LED4
Routing:
- net +3.3V: track 0.00 -> 88.3 mm, vias 0 -> 25
- net /Motor Control Left/~{SLEEP}: track 0.00 -> 58.6 mm, vias 0 -> 3
- net /SPI_MOSI: track 0.00 -> 42.0 mm, vias 0 -> 2
- net /uC/~{RST}: track 0.00 -> 38.8 mm, vias 0 -> 2
- net /SPI_MISO: track 0.00 -> 37.9 mm, vias 0 -> 2
- net GND: track 0.00 -> 32.6 mm, vias 0 -> 304
- net /SPI_CLK: track 0.00 -> 31.6 mm, vias 0 -> 2
- net /uC/SWCLK: track 0.00 -> 31.1 mm, vias 0 -> 2
- net /uC/SWDIO: track 0.00 -> 30.8 mm, vias 0 -> 2
- net /uC/UART_TX: track 0.00 -> 29.7 mm, vias 0 -> 2
- net /uC/~{QSPI_CS}: track 0.00 -> 29.5 mm, vias 0 -> 2
- net /uC/QSPI_IO2: track 0.00 -> 26.2 mm, vias 0 -> 2
- net /uC/QSPI_IO3: track 0.00 -> 25.5 mm, vias 0 -> 2
- net /uC/D-: track 0.00 -> 24.0 mm
- net /uC/LED4: track 0.00 -> 23.4 mm
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- added copper zone on In6.Cu, net +3.3V
- added copper zone on B.Cu, net +BATT
- added copper zone on F.Cu, net +BATT
- added copper zone on F.Cu, net /M_LEFT+
- added copper zone on F.Cu, net /M_LEFT-
- added copper zone on F.Cu, net /M_RIGHT+
- added copper zone on F.Cu, net /M_RIGHT-
- added copper zone on F.Cu, net /VBUS
- added copper zone on In2.Cu, net /VBUS
- added copper zone on F.Cu, net /VBUSFUSE
- added copper zone on F.Cu, net /VCONN
- added copper zone on F.Cu, net /VFUSE
- added copper zone on B.Cu, net GND
- added copper zone on F.Cu, net GND
- added copper zone on In1.Cu, net GND
- added copper zone on In2.Cu, net GND
- added copper zone on In3.Cu, net GND
- added copper zone on In4.Cu, net GND
- added copper zone on In5.Cu, net GND
Other:
- board text added: "3.3V"
- board text added: "BATT"
- board text added: "LED1"
- board text added: "LED2"
- board text added: "LED3"
- board text added: "LED4"

Commit message: tuned lenghts of signals with higher frequencies
Routing:
- net /uC/QSPI_IO1: track 15.6 -> 28.9 mm
- net /SPI_MISO: track 37.9 -> 50.6 mm
- net /SPI_CLK: track 31.6 -> 44.4 mm
- net /uC/QSPI_IO0: track 18.5 -> 28.8 mm
- net /uC/QSPI_CLK: track 20.4 -> 28.9 mm
- net /SPI_MOSI: track 42.0 -> 47.3 mm
- net /uC/QSPI_IO3: track 25.5 -> 29.0 mm
- net /uC/~{QSPI_CS}: track 29.5 -> 32.8 mm
- net /uC/QSPI_IO2: track 26.2 -> 29.0 mm
- net GND: track 32.6 -> 30.7 mm, vias 304 -> 305
- net /uC/D+: track 23.3 -> 24.0 mm

Commit message: firmware - added common classes
Changed lines of the file:
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@@
     (fp_line (start 1.6 0.8) (end -1.6 0.8)
       (stroke (width 0.1) (type solid)) (layer "F.Fab"))
-    (pad "1" smd roundrect (at -1.575 0) (size 1.05 1.9) (layers "F.Cu" "F.Paste" "F.Mask") (roundrect_rratio 0.238095)
+    (pad "1" smd roundrect (at -1.575 0) (size 1.05 1.9) (layers "F.Cu" "F.Paste" "F.Mask") (roundrect_rratio 0.2380952381)
       (net 6 "+3.3V") (pintype "passive"))
-    (pad "2" smd roundrect (at 1.575 0) (size 1.05 1.9) (layers "F.Cu" "F.Paste" "F.Mask") (roundrect_rratio 0.238095)
+    (pad "2" smd roundrect (at 1.575 0) (size 1.05 1.9) (layers "F.Cu" "F.Paste" "F.Mask") (roundrect_rratio 0.2380952381)
       (net 7 "/uC/VREF+") (pintype "passive"))
     (model "${KICAD6_3DMODEL_DIR}/Inductor_SMD.3dshapes/L_1206_3216Metric.wrl"
@@
     (pad "6" smd roundrect locked (at 2.5 1.325 270) (size 0.6 1.55) (layers "F.Cu" "F.Paste" "F.Mask") (roundrect_rratio 0.25)
       (net 3 "GND") (pinfunction "Pin_6") (pintype "passive"))
-    (pad "MP" smd roundrect locked (at -3.8 -1.2 270) (size 1.2 1.8) (layers "F.Cu" "F.Paste" "F.Mask") (roundrect_rratio 0.208333))
-    (pad "MP" smd roundrect locked (at 3.8 -1.2 270) (size 1.2 1.8) (layers "F.Cu" "F.Paste" "F.Mask") (roundrect_rratio 0.208333))
+    (pad "MP" smd roundrect locked (at -3.8 -1.2 270) (size 1.2 1.8) (layers "F.Cu" "F.Paste" "F.Mask") (roundrect_rratio 0.2083333333))
+    (pad "MP" smd roundrect locked (at 3.8 -1.2 270) (size 1.2 1.8) (layers "F.Cu" "F.Paste" "F.Mask") (roundrect_rratio 0.2083333333))
     (model "${KICAD6_3DMODEL_DIR}/Connector_JST.3dshapes/JST_SH_BM06B-SRSS-TB_1x06-1MP_P1.00mm_Vertical.wrl"
       (offset (xyz 0 0 0))
@@
     (pad "6" smd roundrect locked (at 2.5 1.325 90) (size 0.6 1.55) (layers "F.Cu" "F.Paste" "F.Mask") (roundrect_rratio 0.25)
       (net 3 "GND") (pinfunction "Pin_6") (pintype "passive"))
-    (pad "MP" smd roundrect locked (at -3.8 -1.2 90) (size 1.2 1.8) (layers "F.Cu" "F.Paste" "F.Mask") (roundrect_rratio 0.208333))
-    (pad "MP" smd roundrect locked (at 3.8 -1.2 90) (size 1.2 1.8) (layers "F.Cu" "F.Paste" "F.Mask") (roundrect_rratio 0.208333))
+    (pad "MP" smd roundrect locked (at -3.8 -1.2 90) (size 1.2 1.8) (layers "F.Cu" "F.Paste" "F.Mask") (roundrect_rratio 0.2083333333))
+    (pad "MP" smd roundrect locked (at 3.8 -1.2 90) (size 1.2 1.8) (layers "F.Cu" "F.Paste" "F.Mask") (roundrect_rratio 0.2083333333))
     (model "${KICAD6_3DMODEL_DIR}/Connector_JST.3dshapes/JST_SH_BM06B-SRSS-TB_1x06-1MP_P1.00mm_Vertical.wrl"
       (offset (xyz 0 0 0))
@@
     (fp_line (start 7.45 3.4) (end 7.45 -2.35)
       (stroke (width 0.1) (type solid)) (layer "F.Fab"))
-    (pad "1" thru_hole roundrect locked (at 0 0 270) (size 1.7 1.95) (drill 0.95) (layers "*.Cu" "*.Mask") (roundrect_rratio 0.147059)
+    (pad "1" thru_hole roundrect locked (at 0 0 270) (size 1.7 1.95) (drill 0.95) (layers "*.Cu" "*.Mask") (roundrect_rratio 0.1470588235)
       (net 61 "/VCONN") (pinfunction "Pin_1") (pintype "passive"))
     (pad "2" thru_hole oval locked (at 2.5 0 270) (size 1.7 1.95) (drill 0.95) (layers "*.Cu" "*.Mask")
